Commit message: Uniformed naming and urdf tags

File: leg_right.urdf (robot description, URDF)
Before this commit: robot right_leg, 7 links, 6 joints
Links:
- link coxa: geometry collision mesh filename=meshes/coxa_right.stl scale=0.001 0.001 0.001; visual mesh filename=meshes/coxa_right.stl scale=0.001 0.001 0.001
- link femur: geometry collision mesh filename=meshes/femur_right.stl scale=0.001 0.001 0.001; visual mesh filename=meshes/femur_right.stl scale=0.001 0.001 0.001
- link tibia: geometry collision mesh filename=meshes/tibia_right.stl scale=0.001 0.001 0.001; visual mesh filename=meshes/tibia_right.stl scale=0.001 0.001 0.001
Joints:
- joint femur_joint: limit lower=-0.785398 upper=2.356194 effort=1000000 velocity=1000000 -> lower=0 upper=2.356194 effort=1000000 velocity=1000000
