Commit message: Updated hexapod.urdf

File: hexapod.urdf (robot description, URDF)
Before this commit: robot hexapod, 7 links, 6 joints
Links:
- added link leg1_MG996f, mass 0.20641808912389753; collision mesh filename=meshes/MG996.stl scale=0.001 0.001 0.001; visual mesh filename=meshes/MG996.stl scale=0.001 0.001 0.001
- added link leg1_MG996t, mass 0.20641808912389753; collision mesh filename=meshes/MG996.stl scale=0.001 0.001 0.001; visual mesh filename=meshes/MG996.stl scale=0.001 0.001 0.001
- added link leg1_coxa, mass 0.07898637744159479; collision mesh filename=meshes/coxa_right.stl scale=0.001 0.001 0.001; visual mesh filename=meshes/coxa_right.stl scale=0.001 0.001 0.001
- added link leg1_femur, mass 0.2061355014221324; collision mesh filename=meshes/femur_right.stl scale=0.001 0.001 0.001; visual mesh filename=meshes/femur_right.stl scale=0.001 0.001 0.001
- added link leg1_shield, mass 0.09400422482344938; collision mesh filename=meshes/shield.stl scale=0.001 0.001 0.001; visual mesh filename=meshes/shield.stl scale=0.001 0.001 0.001
- added link leg1_tibia, mass 0.09285304614043148; collision mesh filename=meshes/tibia_right.stl scale=0.001 0.001 0.001; visual mesh filename=meshes/tibia_right.stl scale=0.001 0.001 0.001
- added link leg2_MG996f, mass 0.20641808912389753; collision mesh filename=meshes/MG996.stl scale=0.001 0.001 0.001; visual mesh filename=meshes/MG996.stl scale=0.001 0.001 0.001
- added link leg2_MG996t, mass 0.20641808912389753; collision mesh filename=meshes/MG996.stl scale=0.001 0.001 0.001; visual mesh filename=meshes/MG996.stl scale=0.001 0.001 0.001
- added link leg2_coxa, mass 0.07898637744159479; collision mesh filename=meshes/coxa_right.stl scale=0.001 0.001 0.001; visual mesh filename=meshes/coxa_right.stl scale=0.001 0.001 0.001
- added link leg2_femur, mass 0.2061355014221324; collision mesh filename=meshes/femur_right.stl scale=0.001 0.001 0.001; visual mesh filename=meshes/femur_right.stl scale=0.001 0.001 0.001
- added link leg2_shield, mass 0.09400422482344938; collision mesh filename=meshes/shield.stl scale=0.001 0.001 0.001; visual mesh filename=meshes/shield.stl scale=0.001 0.001 0.001
- added link leg2_tibia, mass 0.09285304614043148; collision mesh filename=meshes/tibia_right.stl scale=0.001 0.001 0.001; visual mesh filename=meshes/tibia_right.stl scale=0.001 0.001 0.001
- added link leg3_MG996f, mass 0.20641808912389753; collision mesh filename=meshes/MG996.stl scale=0.001 0.001 0.001; visual mesh filename=meshes/MG996.stl scale=0.001 0.001 0.001
- added link leg3_MG996t, mass 0.20641808912389753; collision mesh filename=meshes/MG996.stl scale=0.001 0.001 0.001; visual mesh filename=meshes/MG996.stl scale=0.001 0.001 0.001
- added link leg3_coxa, mass 0.07898637744159479; collision mesh filename=meshes/coxa_right.stl scale=0.001 0.001 0.001; visual mesh filename=meshes/coxa_right.stl scale=0.001 0.001 0.001
- added link leg3_femur, mass 0.2061355014221324; collision mesh filename=meshes/femur_right.stl scale=0.001 0.001 0.001; visual mesh filename=meshes/femur_right.stl scale=0.001 0.001 0.001
- added link leg3_shield, mass 0.09400422482344938; collision mesh filename=meshes/shield.stl scale=0.001 0.001 0.001; visual mesh filename=meshes/shield.stl scale=0.001 0.001 0.001
- added link leg3_tibia, mass 0.09285304614043148; collision mesh filename=meshes/tibia_right.stl scale=0.001 0.001 0.001; visual mesh filename=meshes/tibia_right.stl scale=0.001 0.001 0.001
- added link leg4_MG996f, mass 0.20641808912389753; collision mesh filename=meshes/MG996.stl scale=0.001 0.001 0.001; visual mesh filename=meshes/MG996.stl scale=0.001 0.001 0.001
- added link leg4_MG996t, mass 0.20641808912389753; collision mesh filename=meshes/MG996.stl scale=0.001 0.001 0.001; visual mesh filename=meshes/MG996.stl scale=0.001 0.001 0.001
- added link leg4_coxa, mass 0.07898637744159481; collision mesh filename=meshes/coxa_left.stl scale=0.001 0.001 0.001; visual mesh filename=meshes/coxa_left.stl scale=0.001 0.001 0.001
- added link leg4_femur, mass 0.2061355014221325; collision mesh filename=meshes/femur_left.stl scale=0.001 0.001 0.001; visual mesh filename=meshes/femur_left.stl scale=0.001 0.001 0.001
- added link leg4_shield, mass 0.09400422482344938; collision mesh filename=meshes/shield.stl scale=0.001 0.001 0.001; visual mesh filename=meshes/shield.stl scale=0.001 0.001 0.001
- added link leg4_tibia, mass 0.09285304614043133; collision mesh filename=meshes/tibia_left.stl scale=0.001 0.001 0.001; visual mesh filename=meshes/tibia_left.stl scale=0.001 0.001 0.001
- added link leg5_MG996f, mass 0.20641808912389753; collision mesh filename=meshes/MG996.stl scale=0.001 0.001 0.001; visual mesh filename=meshes/MG996.stl scale=0.001 0.001 0.001
- added link leg5_MG996t, mass 0.20641808912389753; collision mesh filename=meshes/MG996.stl scale=0.001 0.001 0.001; visual mesh filename=meshes/MG996.stl scale=0.001 0.001 0.001
- added link leg5_coxa, mass 0.07898637744159481; collision mesh filename=meshes/coxa_left.stl scale=0.001 0.001 0.001; visual mesh filename=meshes/coxa_left.stl scale=0.001 0.001 0.001
- added link leg5_femur, mass 0.2061355014221325; collision mesh filename=meshes/femur_left.stl scale=0.001 0.001 0.001; visual mesh filename=meshes/femur_left.stl scale=0.001 0.001 0.001
- added link leg5_shield, mass 0.09400422482344938; collision mesh filename=meshes/shield.stl scale=0.001 0.001 0.001; visual mesh filename=meshes/shield.stl scale=0.001 0.001 0.001
- added link leg5_tibia, mass 0.09285304614043133; collision mesh filename=meshes/tibia_left.stl scale=0.001 0.001 0.001; visual mesh filename=meshes/tibia_left.stl scale=0.001 0.001 0.001
- added link leg6_MG996f, mass 0.20641808912389753; collision mesh filename=meshes/MG996.stl scale=0.001 0.001 0.001; visual mesh filename=meshes/MG996.stl scale=0.001 0.001 0.001
- added link leg6_MG996t, mass 0.20641808912389753; collision mesh filename=meshes/MG996.stl scale=0.001 0.001 0.001; visual mesh filename=meshes/MG996.stl scale=0.001 0.001 0.001
- added link leg6_coxa, mass 0.07898637744159481; collision mesh filename=meshes/coxa_left.stl scale=0.001 0.001 0.001; visual mesh filename=meshes/coxa_left.stl scale=0.001 0.001 0.001
- added link leg6_femur, mass 0.2061355014221325; collision mesh filename=meshes/femur_left.stl scale=0.001 0.001 0.001; visual mesh filename=meshes/femur_left.stl scale=0.001 0.001 0.001
- added link leg6_shield, mass 0.09400422482344938; collision mesh filename=meshes/shield.stl scale=0.001 0.001 0.001; visual mesh filename=meshes/shield.stl scale=0.001 0.001 0.001
- added link leg6_tibia, mass 0.09285304614043133; collision mesh filename=meshes/tibia_left.stl scale=0.001 0.001 0.001; visual mesh filename=meshes/tibia_left.stl scale=0.001 0.001 0.001
Joints:
- added joint leg1_MG996t_tibia: type fixed, parent leg1_MG996t, child leg1_tibia, origin xyz=0.0024041599999999976 -0.018031230000000013 0.005250000000000004 rpy=-3.141592653589793 -5.55111512312578e-17 0.0
- added joint leg1_coxa_MG996f: type fixed, parent leg1_coxa, child leg1_MG996f, origin xyz=-0.02916816000000001 -0.03906765 -0.04585 rpy=-0.0 -1.5707963267948966 0
- added joint leg1_coxa_joint: type revolute, parent leg1_MG996c, child leg1_coxa, origin xyz=-0.028425689999999997 0.021001069999999997 -0.01005 rpy=3.141592653589793 -0.0 0.0, axis 0.0 0.0 1.0, limit lower=-1.570796 upper=1.570796 effort=1000000 velocity=1000000
- added joint leg1_femur_joint: type revolute, parent leg1_MG996f, child leg1_femur, origin xyz=0.03495 -0.0033941100000000014 -0.010818740000000009 rpy=-0.0 1.5707963267948966 0, axis 0.707107 -0.707107 0.0, limit lower=-0.785398 upper=2.356194 effort=1000000 velocity=1000000
- added joint leg1_tibia_joint: type revolute, parent leg1_femur, child leg1_MG996t, origin xyz=-0.020211430000000002 -0.021625650000000007 0.06344155000000001 rpy=3.141592653589793 -5.551115123125783e-17 0.0, axis 0.707107 0.707107 3.925232361368103e-17, limit lower=0.0 upper=1.570796 effort=1000000 velocity=1000000
- added joint leg1_tibia_shield: type fixed, parent leg1_tibia, child leg1_shield, origin xyz=-0.07392547999999997 -0.05794487000000002 0.02125 rpy=-3.222902565236662e-64 -1.5707963267948966 0
- added joint leg2_MG996f_Rigido-18: type fixed, parent leg2_MG996f, child leg2_tibia, origin xyz=0.014450000000000003 -0.01105 -0.005250000000000004 rpy=-3.141592653589793 -1.2516661846134429e-49 0.0
- added joint leg2_MG996t_Rivoluzione-16: type revolute, parent leg2_MG996t, child leg2_femur, origin xyz=0.03495 -0.010050000000000002 -0.005250000000000004 rpy=-0.0 1.5707963267948966 0, axis 0.0 -1.0 0.0, limit lower=-0.785398 upper=2.356194 effort=1000000 velocity=1000000
- added joint leg2_coxa_MG996f: type fixed, parent leg2_coxa, child leg2_MG996t, origin xyz=-0.048249999999999994 -0.006999999999999999 -0.04585 rpy=-0.0 -1.5707963267948966 0
- added joint leg2_coxa_joint: type revolute, parent leg2_MG996c, child leg2_coxa, origin xyz=-0.03495 -0.00525 -0.01005 rpy=3.141592653589793 -0.0 0.0, axis 0.0 0.0 1.0, limit lower=-1.570796 upper=1.570796 effort=1000000 velocity=1000000
- added joint leg2_femur_Rivoluzione-17: type revolute, parent leg2_femur, child leg2_MG996f, origin xyz=-0.029583280000000017 -0.0009999999999999987 0.06344155000000001 rpy=3.141592653589793 -0.0 0.0, axis 0.0 1.0 0.0, limit lower=0.0 upper=1.570796 effort=1000000 velocity=1000000
- added joint leg2_tibia_Rigido-19: type fixed, parent leg2_tibia, child leg2_shield, origin xyz=-0.09324641 0.0113 0.010749999999999994 rpy=-0.0 -1.5707963267948966 0
- added joint leg3_MG996c_Rivoluzione-20: type revolute, parent leg3_MG996c, child leg3_coxa, origin xyz=-0.021001069999999997 -0.028425690000000003 -0.01005 rpy=3.141592653589793 -0.0 0.0, axis 0.0 0.0 1.0, limit lower=-1.570796 upper=1.570796 effort=1000000 velocity=1000000
- added joint leg3_MG996f_Rivoluzione-22: type revolute, parent leg3_MG996f, child leg3_femur, origin xyz=0.03495 -0.010818740000000009 0.0033941100000000014 rpy=-0.0 1.5707963267948966 0, axis -0.707107 -0.707107 0.0, limit lower=-0.785398 upper=2.356194 effort=1000000 velocity=1000000
- added joint leg3_MG996t_Rigido-24: type fixed, parent leg3_MG996t, child leg3_tibia, origin xyz=0.017324120000000002 -0.0031112699999999906 -0.0052500000000000125 rpy=0.0 -3.050517397236834e-32 1.3465939511877539e-48
- added joint leg3_coxa_Rigido-21: type fixed, parent leg3_coxa, child leg3_MG996f, origin xyz=-0.03906765 0.02916816000000001 -0.04585 rpy=-0.0 -1.5707963267948966 0
- added joint leg3_femur_Rivoluzione-23: type revolute, parent leg3_femur, child leg3_MG996t, origin xyz=-0.02268630999999999 0.01915077 0.06344155000000001 rpy=0.0 -0.0 0.0, axis 0.707107 0.7071069999999999 -6.483768997034379e-17, limit lower=-1.570796 upper=0.0 effort=1000000 velocity=1000000
- added joint leg3_tibia_Rigido-25: type fixed, parent leg3_tibia, child leg3_shield, origin xyz=-0.05794486000000001 0.07392547999999997 0.02125 rpy=4.930380657631325e-32 -1.5707963267948966 0
- added joint leg4_MG996c_Rivoluzione-26: type revolute, parent leg4_MG996c, child leg4_coxa, origin xyz=0.028425689999999997 -0.021001069999999997 -0.01005 rpy=3.141592653589793 -0.0 0.0, axis 0.0 0.0 1.0, limit lower=-1.570796 upper=1.570796 effort=1000000 velocity=1000000
- added joint leg4_MG996f_Rivoluzione-28: type revolute, parent leg4_MG996f, child leg4_femur, origin xyz=-0.014450000000000001 0.0033941100000000014 0.010818729999999999 rpy=3.141592653589793 -1.5707963267948966 0, axis 0.707107 -0.7071069999999999 -4.6222332968741714e-33, limit lower=-2.356194 upper=0.785398 effort=1000000 velocity=1000000
- added joint leg4_MG996t_Rigido-30: type fixed, parent leg4_MG996t, child leg4_tibia, origin xyz=-0.018031230000000013 0.0024041600000000154 0.005250000000000004 rpy=-3.141592653589793 -5.592845782213225e-17 -4.850773625799853e-32
- added joint leg4_coxa_Rigido-27: type fixed, parent leg4_coxa, child leg4_MG996f, origin xyz=0.03164303 0.02174353 0.0027500000000000037 rpy=-3.141592653589793 -1.5707963267948966 0
- added joint leg4_femur_Rivoluzione-29: type revolute, parent leg4_femur, child leg4_MG996t, origin xyz=0.021625650000000007 0.020211430000000002 0.06344155 rpy=3.141592653589793 -5.592845782213251e-17 -3.655944291150896e-49, axis -0.7071069999999999 -0.7071069999999999 -3.228531091625886e-17, limit lower=0.0 upper=1.570796 effort=1000000 velocity=1000000
- added joint leg4_tibia_Rigido-31: type fixed, parent leg4_tibia, child leg4_shield, origin xyz=0.05794487000000002 0.07392548000000002 0.02124999999999999 rpy=3.141592653589793 -1.5707963267948966 0
- added joint leg5_MG996c_Rivoluzione-32: type revolute, parent leg5_MG996c, child leg5_coxa, origin xyz=0.03495 0.00525 -0.01005 rpy=3.141592653589793 -0.0 0.0, axis 0.0 0.0 1.0, limit lower=-1.570796 upper=1.570796 effort=1000000 velocity=1000000
- added joint leg5_MG996f_Rivoluzione-34: type revolute, parent leg5_MG996f, child leg5_femur, origin xyz=0.03495 0.010050000000000002 0.005249999999999986 rpy=-3.141592653589793 -1.5707963267948966 0, axis 0.0 -1.0 0.0, limit lower=-2.356194 upper=0.785398 effort=1000000 velocity=1000000
- added joint leg5_MG996t_Rigido-36: type fixed, parent leg5_MG996t, child leg5_tibia, origin xyz=-0.014450000000000003 -0.01105 -0.005250000000000004 rpy=3.141592653589793 -3.627598386426413e-33 8.086363567567113e-66
- added joint leg5_coxa_Rigido-33: type fixed, parent leg5_coxa, child leg5_MG996f, origin xyz=0.037750000000000006 -0.006999999999999999 -0.04585 rpy=-3.141592653589793 -1.5707963267948966 0
- added joint leg5_femur_Rivoluzione-35: type revolute, parent leg5_femur, child leg5_MG996t, origin xyz=0.029583280000000017 -0.0009999999999999987 0.06344155000000001 rpy=-3.141592653589793 -3.627598386426402e-33 0.0, axis 0.0 -1.0 2.229123157024303e-33, limit lower=0.0 upper=1.570796 effort=1000000 velocity=1000000
- added joint leg5_tibia_Rigido-37: type fixed, parent leg5_tibia, child leg5_shield, origin xyz=0.09324640999999999 0.0113 0.010749999999999994 rpy=3.141592653589793 -1.5707963267948966 0
- added joint leg6_MG996c_Rivoluzione-38: type revolute, parent leg6_MG996c, child leg6_coxa, origin xyz=0.021001069999999997 0.028425690000000003 -0.01005 rpy=3.141592653589793 -0.0 0.0, axis 0.0 0.0 1.0, limit lower=-1.570796 upper=1.570796 effort=1000000 velocity=1000000
- added joint leg6_MG996f_Rivoluzione-40: type revolute, parent leg6_MG996f, child leg6_femur, origin xyz=0.03495 0.010818729999999999 -0.0033941100000000014 rpy=-3.141592653589793 -1.5707963267948966 0, axis -0.707107 -0.7071070000000002 0.0, limit lower=-2.356194 upper=0.785398 effort=1000000 velocity=1000000
- added joint leg6_MG996t_Rigido-42: type fixed, parent leg6_MG996t, child leg6_tibia, origin xyz=-0.0024041599999999976 -0.018031230000000013 0.005250000000000004 rpy=3.141592653589793 -0.0 -5.55111512312578e-17
- added joint leg6_coxa_Rigido-39: type fixed, parent leg6_coxa, child leg6_MG996f, origin xyz=0.02174353 -0.03164303 -0.04585 rpy=-3.141592653589793 -1.5707963267948966 0
- added joint leg6_femur_Rivoluzione-41: type revolute, parent leg6_femur, child leg6_MG996t, origin xyz=0.020211430000000002 -0.02162564999999999 0.06344154999999999 rpy=3.141592653589793 -0.0 -5.5511151231257815e-17, axis 0.707107 -0.707107 0.0, limit lower=0.0 upper=1.570796 effort=1000000 velocity=1000000
- added joint leg6_tibia_Rigido-43: type fixed, parent leg6_tibia, child leg6_shield, origin xyz=0.07392547999999997 -0.05794487000000002 0.02125 rpy=-3.141592653589793 -1.5707963267948966 0
