Commit message: Updated input data (URDF, config)

File: data/URDF/hexapod.urdf (robot description, URDF)
Before this commit: robot hexapod, 43 links, 42 joints
Links:
- removed link leg1_shield
- removed link leg2_shield
- removed link leg3_shield
- removed link leg4_shield
- removed link leg5_shield
- removed link leg6_shield
Joints:
- removed joint leg1_tibia_shield
- removed joint leg2_tibia_shield
- removed joint leg3_tibia_shield
- removed joint leg4_tibia_shield
- removed joint leg5_tibia_shield
- removed joint leg6_tibia_shield
- joint leg1_tibia_joint: limit lower=0.0 upper=1.570796 effort=1000000 velocity=1000000 -> lower=-3.14159 upper=3.14159 effort=1000000 velocity=1000000
- joint leg2_tibia_joint: limit lower=0.0 upper=1.570796 effort=1000000 velocity=1000000 -> lower=-3.14159 upper=3.14159 effort=1000000 velocity=1000000
- joint leg3_tibia_joint: limit lower=0.0 upper=1.570796 effort=1000000 velocity=1000000 -> lower=-3.14159 upper=3.14159 effort=1000000 velocity=1000000
- joint leg4_tibia_joint: limit lower=0.0 upper=1.570796 effort=1000000 velocity=1000000 -> lower=-3.14159 upper=3.14159 effort=1000000 velocity=1000000
- joint leg5_tibia_joint: limit lower=0.0 upper=1.570796 effort=1000000 velocity=1000000 -> lower=-3.14159 upper=3.14159 effort=1000000 velocity=1000000
- joint leg6_tibia_joint: limit lower=0.0 upper=1.570796 effort=1000000 velocity=1000000 -> lower=-3.14159 upper=3.14159 effort=1000000 velocity=1000000
